File: hardware/irin.kicad_sch (KiCad schematic)
At the start: 12 parts, among them J1 Battery terminals, J2 DHT22 remote (VCC/DATA/GND), U1 MP1584EN set to 5.0V, U2 01Space ESP32-C3-0.42LCD, U3 HiLetgo ADS1115 (0x48, ADDR->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

Commit message: Rename project to Irin
Irin (Aramaic ʿirin, "watchers", "the wakeful ones") from the Book of
Enoch; the name's root is documented in README.md and CLAUDE.md.

- KiCad project hardware/irin.*, footprint library Uncharted -> Irin;
  ERC unchanged, regenerated netlist equivalent, preview.pdf refreshed
- Firmware config esphome/irin.yaml, dashboard ha_config/dashboard.yaml
- Breadboard generator points at irin.net; regenerated, validates OK
- The "Uncharted 12V" instance keeps its device name, entity IDs and
  secrets keys so existing HA entities and history are untouched

Co-Authored-By: Claude Opus 5.5 <noreply@anthropic.com>
Parts:
- C1, C3: symbol Uncharted:C -> Irin:C
- C2: symbol Uncharted:CP -> Irin:CP
- D1: symbol Uncharted:TVS -> Irin:TVS
- F1: symbol Uncharted:FUSE -> Irin:FUSE
- J1: symbol Uncharted:BATT_CONN -> Irin:BATT_CONN
- J2: symbol Uncharted:DHT22 -> Irin:DHT22
- R1, R2: symbol Uncharted:R -> Irin:R
- U1: footprint Uncharted:MP1584EN_HW133_2x2Pad_P2.54mm_W7.62mm_L17.78mm -> Irin:MP1584EN_HW133_2x2Pad_P2.54mm_W7.62mm_L17.78mm; symbol Uncharted:BUCK_MODULE -> Irin:BUCK_MODULE
- U2: footprint Uncharted:ESP32C3_042LCD_2x8_P2.54mm_W17.78mm -> Irin:ESP32C3_042LCD_2x8_P2.54mm_W17.78mm; symbol Uncharted:ESP32C3_BOARD -> Irin:ESP32C3_BOARD
- U3: footprint Uncharted:ADS1115_HiLetgo_1x10_P2.54mm_W18mm_L28.3mm -> Irin:ADS1115_HiLetgo_1x10_P2.54mm_W18mm_L28.3mm; symbol Uncharted:ADS1115 -> Irin:ADS1115
Other:
- title: Uncharted 12V Battery Monitor -> Irin — 12V Battery Monitor
Changed lines of the file:
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@@
 	(paper "A2")
 	(title_block
-		(title "Uncharted 12V Battery Monitor")
+		(title "Irin — 12V Battery Monitor")
 		(date "2026-08-29")
 		(rev "B")
 		(company "Owner-built")
-		(comment 1 "ESP32-C3 + ADS1115 12V battery monitor for 2027 Subaru Uncharted GT")
+		(comment 1 "ESP32-C3 + ADS1115 battery monitor. Prototype: 2027 Subaru Uncharted GT")
 		(comment 2 "See CLAUDE.md / PARTS.md in project root for full design rationale")
 	)
@@
 	)
 	(symbol
-		(lib_id "Uncharted:R")
+		(lib_id "Irin:R")
 		(at 129.54 134.62 270)
 		(unit 1)
@@
 		)
 		(instances
-			(project "uncharted-battery-monitor"
+			(project "irin"
 				(path "/097d63fa-dc7b-4932-a049-360b053b132d"
 					(reference "R2")
@@
 	)
 	(symbol
-		(lib_id "Uncharted:CP")
+		(lib_id "Irin:CP")
 		(at 180.34 95.25 270)
 		(unit 1)
@@
 		)
 		(instances
-			(project "uncharted-battery-monitor"
+			(project "irin"
 				(path "/097d63fa-dc7b-4932-a049-360b053b132d"
 					(reference "C2")
@@
 	)
 	(symbol
-		(lib_id "Uncharted:R")
+		(lib_id "Irin:R")
 		(at 129.54 64.77 270)
 		(unit 1)
@@
 		)
 		(instances
-			(project "uncharted-battery-monitor"
+			(project "irin"
 				(path "/097d63fa-dc7b-4932-a049-360b053b132d"
 					(reference "R1")
@@
 	)
 	(symbol
-		(lib_id "Uncharted:ESP32C3_BOARD")
+		(lib_id "Irin:ESP32C3_BOARD")
 		(at 299.72 90.17 0)
 		(unit 1)
@@
 			)
 		)
-		(property "Footprint" "Uncharted:ESP32C3_042LCD_2x8_P2.54mm_W17.78mm"
+		(property "Footprint" "Irin:ESP32C3_042LCD_2x8_P2.54mm_W17.78mm"
 			(at 299.72 90.17 0)
 			(hide yes)
@@
 		)
 		(instances
-			(project "uncharted-battery-monitor"
+			(project "irin"
 				(path "/097d63fa-dc7b-4932-a049-360b053b132d"
 					(reference "U2")
@@
 	)
 	(symbol
-		(lib_id "Uncharted:TVS")
+		(lib_id "Irin:TVS")
 		(at 95.25 95.25 270)
 		(unit 1)
@@
 		)
 		(instances
-			(project "uncharted-battery-monitor"
+			(project "irin"
 				(path "/097d63fa-dc7b-4932-a049-360b053b132d"
 					(reference "D1")
@@
 	)
 	(symbol
-		(lib_id "Uncharted:C")
+		(lib_id "Irin:C")
 		(at 199.39 95.25 270)
 		(unit 1)
@@
 		)
 		(instances
-			(project "uncharted-battery-monitor"
+			(project "irin"
 				(path "/097d63fa-dc7b-4932-a049-360b053b132d"
 					(reference "C3")
@@
 	)
 	(symbol
-		(lib_id "Uncharted:ADS1115")
+		(lib_id "Irin:ADS1115")
 		(at 359.41 54.61 0)
 		(unit 1)
@@
 			)
 		)
-		(property "Footprint" "Uncharted:ADS1115_HiLetgo_1x10_P2.54mm_W18mm_L28.3mm"
+		(property "Footprint" "Irin:ADS1115_HiLetgo_1x10_P2.54mm_W18mm_L28.3mm"
 			(at 359.41 54.61 0)
 			(hide yes)
@@
 		)
 		(instances
-			(project "uncharted-battery-monitor"
+			(project "irin"
 				(path "/097d63fa-dc7b-4932-a049-360b053b132d"
 					(reference "U3")
@@
 	)
 	(symbol
-		(lib_id "Uncharted:DHT22")
+		(lib_id "Irin:DHT22")
 		(at 359.41 139.7 0)
 		(unit 1)
@@
 		)
 		(instances
-			(project "uncharted-battery-monitor"
+			(project "irin"
 				(path "/097d63fa-dc7b-4932-a049-360b053b132d"
 					(reference "J2")
@@
 	)
 	(symbol
-		(lib_id "Uncharted:FUSE")
+		(lib_id "Irin:FUSE")
 		(at 62.23 100.33 0)
 		(unit 1)
@@
 		)
 		(instances
-			(project "uncharted-battery-monitor"
+			(project "irin"
 				(path "/097d63fa-dc7b-4932-a049-360b053b132d"
 					(reference "F1")
@@
 	)
 	(symbol
-		(lib_id "Uncharted:C")
+		(lib_id "Irin:C")
 		(at 154.94 134.62 270)
 		(unit 1)
@@
 		)
 		(instances
-			(project "uncharted-battery-monitor"
+			(project "irin"
 				(path "/097d63fa-dc7b-4932-a049-360b053b132d"
 					(reference "C1")
@@
 	)
 	(symbol
-		(lib_id "Uncharted:BUCK_MODULE")
+		(lib_id "Irin:BUCK_MODULE")
 		(at 245.11 90.17 0)
 		(unit 1)
@@
 			)
 		)
-		(property "Footprint" "Uncharted:MP1584EN_HW133_2x2Pad_P2.54mm_W7.62mm_L17.78mm"
+		(property "Footprint" "Irin:MP1584EN_HW133_2x2Pad_P2.54mm_W7.62mm_L17.78mm"
 			(at 245.11 90.17 0)
 			(hide yes)
@@
 		)
 		(instances
-			(project "uncharted-battery-monitor"
+			(project "irin"
 				(path "/097d63fa-dc7b-4932-a049-360b053b132d"
 					(reference "U1")
@@
 	)
 	(symbol
-		(lib_id "Uncharted:BATT_CONN")
+		(lib_id "Irin:BATT_CONN")
 		(at 20.32 100.33 0)
 		(unit 1)
@@
 		)
 		(instances
-			(project "uncharted-battery-monitor"
+			(project "irin"
 				(path "/097d63fa-dc7b-4932-a049-360b053b132d"
 					(reference "J1")

Commit message: Hardware: conventional schematic symbols; PCB outline, placement, GND plane, routing
Schematic (netlist unchanged):
- ANSI resistors, two-plate caps, TVS with cathode bar, fuse, battery (J1)
- Detailed ESP32-C3, ADS1115 and DHT22 symbols; U2 3V3 top / GND bottom,
  U1 outputs on the right

PCB:
- Board outline 78.5 x 69 mm, four M3 mounting holes inset 3.5 mm
- Parts re-placed, C3 at the buck input, divider beside the ADS1115
- B.Cu GND plane with thermal reliefs; "Pwr" net class (0.4 mm) for 12vPROT
- Fully routed: DRC 0 violations, 0 unconnected, 0 schematic parity issues

Regenerated preview.pdf and irin.net.

Co-Authored-By: Claude Opus 5.5 <noreply@anthropic.com>
Other:
- note added: "TVS D1: P6KE18A, UNIDIRECTIONAL, optional. BANDED END (K, cathode, square pad) to PROT, A (anode) to GND. Reverse-biased in normal service: VRWM 15.3 V, breakdown 17.1-18.9 V, clamps a surge at Vc 25.2 V (MP1584 abs max 30 V). Fitted backwards it is a forward diode across the supply and blows F1."
- note removed: "TVS D1 is P6KE18A UNIDIRECTIONAL, optional. K (cathode) to PROT, A (anode) to GND -- conducts to clamp the rail, like a reverse-biased zener."
- moved on the sheet: C2, U1

Commit message: Hardware rev B: swap buck and ADC sides, reroute, antenna keepout
- U1 (MP1584) and U3 (ADS1115) swapped so each sits beside the U2 pins it
  serves; input parts (J1, D1, C3, C2) moved to the right/top, 12 V now a
  straight drop to U1. All routing on F.Cu; B.Cu is an unbroken GND plane
  apart from a rule-area keepout under U2's antenna end. No vias.
  DRC 0 / unconnected 0 / parity clean.
- Schematic: F1 is the inline harness fuse (excluded from board, kept in
  BOM); BT1 (vehicle battery, off-board) added inside a dashed
  "OFF-BOARD (vehicle harness)" box. J1 redrawn as a 2-pin connector.
  J2 and divider notes updated (DHT22 inside for now; PCB divider ground
  goes straight to the plane). ERC: only the 12 library-config warnings.
- CLAUDE.md: USB-end margin kept for lid-off cable access, antenna end,
  J1 position for the enclosure model.

Co-Authored-By: Claude Opus 5.5 <noreply@anthropic.com>
Parts:
- added BT1: Vehicle 12V (flooded, 50Ah), symbol Device:Battery
- F1: value 5A (Micro2 blade) -> 5A Micro2, inline
Connections:
- net 12vPROT: now also J1.1 (BATT+)
- net GND: now also BT1.2 (-)
- net at F1.1: now also BT1.1 (+); no longer J1.1 (BATT+)
Other:
- note added: "Divider R1 47k / R2 10k = 5.7:1 (unit 1 measured 46.5k/9.85k = 5.72:1). C1 = 2 x 1000pF mica in parallel (2nF, low leakage). ADS1115 abs max = VDD+0.3 = 3.6V. 12.22V(flooded 50% SOC)->2.14V 14.4V(charging)->2.52V 16.0V(design max)->2.80V @ A0. ANALOG GROUND: on the PCB, R2 and C1 return straight to the solid B.Cu GND plane (offset is microvolts). Wired builds: return them to the ADS1115 GND pin, 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"
- note added: "J2: DHT22/AM2302, 1=VCC 2=DATA 3=GND. Data pull-up is on the sensor module. For now the sensor is INSIDE the enclosure, hot-glued to the wall (reads a few degC warm, which errs safe). Remote option: cable out through a gland, max ~1 m at 3.3 V."
- note added: "OFF-BOARD (vehicle harness) F1: inline holder, as close to the battery + terminal as practical."
- note removed: "Divider R1 47k / R2 10k = 5.7:1 (unit 1 measured 46.5k/9.85k = 5.72:1). C1 = 2 x 1000pF mica in parallel (2nF, low leakage). ADS1115 abs max = VDD+0.3 = 3.6V. 12.22V(flooded 50% SOC)->2.14V 14.4V(charging)->2.52V 16.0V(design max)->2.80V @ A0. ANALOG GROUND: R2 and C1 return to the ADS1115 GND pin, and that node meets power GND at ONE point. Load current through a shared ground path adds directly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"
- note removed: "J2: cable to REMOTE DHT22/AM2302, mounted outside the enclosure (via gland). 1=VCC 2=DATA 3=GND. Data pull-up is on the sensor module. At 3.3 V supply, AM2302 datasheet limits cable length to ~1 m."
- moved on the sheet: F1
Changed lines of the file:
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@@
 		)
 	)
-	(text "J2: cable to REMOTE DHT22/AM2302, mounted outside the enclosure (via gland).\n1=VCC 2=DATA 3=GND. Data pull-up is on the sensor module.\nAt 3.3 V supply, AM2302 datasheet limits cable length to ~1 m."
+	(text "J2: DHT22/AM2302, 1=VCC 2=DATA 3=GND. Data pull-up is on the sensor module.\nFor now the sensor is INSIDE the enclosure, hot-glued to the wall (reads a few degC\nwarm, which errs safe). Remote option: cable out through a gland, max ~1 m at 3.3 V."
 		(exclude_from_sim no)
 		(at 355 165 0)
@@
 		)
 	)
-	(text "Divider R1 47k / R2 10k = 5.7:1 (unit 1 measured 46.5k/9.85k = 5.72:1). C1 = 2 x 1000pF mica\nin parallel (2nF, low leakage). ADS1115 abs max = VDD+0.3 = 3.6V.\n12.22V(flooded 50% SOC)->2.14V  14.4V(charging)->2.52V  16.0V(design max)->2.80V @ A0.\nANALOG GROUND: R2 and C1 return to the ADS1115 GND pin, and that node meets power GND\nat ONE point. Load current through a shared ground path adds directly to A0 and is\nscaled up 5.7x (bench: 15mV rail-to-rail = ~86mV error at the battery)."
+	(text "Divider R1 47k / R2 10k = 5.7:1 (unit 1 measured 46.5k/9.85k = 5.72:1). C1 = 2 x 1000pF mica\nin parallel (2nF, low leakage). ADS1115 abs max = VDD+0.3 = 3.6V.\n12.22V(flooded 50% SOC)->2.14V  14.4V(charging)->2.52V  16.0V(design max)->2.80V @ A0.\nANALOG GROUND: on the PCB, R2 and C1 return straight to the solid B.Cu GND plane (offset\nis microvolts). Wired builds: return them to the ADS1115 GND pin, meeting power GND at ONE\npoint (bench: 15mV rail-to-rail drop = ~86mV error at the battery after the 5.7x scale-up)."
 		(exclude_from_sim no)
 		(at 125.476 180.848 0)
@@
 	)
 	(junction
+		(at 59.69 69.85)
+		(diameter 0)
+		(color 0 0 0 0)
+	)
+	(junction
 		(at 129.54 30.48)
 		(diameter 0)
@@
 	)
 	(junction
-		(at 129.54 130.81)
+		(at 95.25 30.48)
 		(diameter 0)
 		(color 0 0 0 0)
 	)
 	(junction
-		(at 95.25 30.48)
+		(at 129.54 130.81)
 		(diameter 0)
 		(color 0 0 0 0)
@@
 	(wire
 		(pts
-			(xy 55.88 100.33) (xy 58.42 100.33)
-		)
-		(stroke
-			(width 0)
-			(type default)
-		)
-	)
-	(wire
-		(pts
 			(xy 129.54 138.43) (xy 129.54 158.75)
 		)
@@
 	(wire
 		(pts
-			(xy 69.85 100.33) (xy 69.85 30.48)
+			(xy 59.69 69.85) (xy 59.69 91.44)
 		)
 		(stroke
@@
 	(wire
 		(pts
-			(xy 16.51 158.75) (xy 95.25 158.75)
+			(xy 59.69 158.75) (xy 95.25 158.75)
 		)
 		(stroke
@@
 	(wire
 		(pts
-			(xy 16.51 99.06) (xy 16.51 95.25)
-		)
-		(stroke
-			(width 0)
-			(type default)
-		)
-	)
-	(wire
-		(pts
 			(xy 129.54 30.48) (xy 180.34 30.48)
 		)
@@
 	(wire
 		(pts
+			(xy 34.29 69.85) (xy 59.69 69.85)
+		)
+		(stroke
+			(width 0)
+			(type default)
+		)
+	)
+	(wire
+		(pts
 			(xy 354.33 101.6) (xy 356.87 101.6)
 		)
@@
 	(wire
 		(pts
-			(xy 16.51 109.22) (xy 16.51 158.75)
-		)
-		(stroke
-			(width 0)
-			(type default)
-		)
-	)
-	(wire
-		(pts
-			(xy 16.51 95.25) (xy 55.88 95.25)
+			(xy 59.69 101.6) (xy 59.69 158.75)
 		)
 		(stroke
@@
 	(wire
 		(pts
-			(xy 69.85 100.33) (xy 66.04 100.33)
-		)
-		(stroke
-			(width 0)
-			(type default)
-		)
-	)
-	(wire
-		(pts
-			(xy 69.85 30.48) (xy 95.25 30.48)
+			(xy 59.69 69.85) (xy 59.69 30.48)
+		)
+		(stroke
+			(width 0)
+			(type default)
+		)
+	)
+	(wire
+		(pts
+			(xy 59.69 30.48) (xy 95.25 30.48)
 		)
 		(stroke
@@
 	(wire
 		(pts
-			(xy 55.88 95.25) (xy 55.88 100.33)
-		)
-		(stroke
-			(width 0)
-			(type default)
-		)
-	)
-	(wire
-		(pts
 			(xy 154.94 158.75) (xy 180.34 158.75)
 		)
@@
 	)
 	(label "GND"
-		(at 16.51 158.75 0)
+		(at 59.69 158.75 0)
 		(effects
 			(font
@@
 	)
 	(label "12vPROT"
-		(at 69.85 30.48 0)
+		(at 59.69 30.48 0)
 		(effects
 			(font
@@
 	(symbol
 		(lib_id "Irin:FUSE")
-		(at 62.23 100.33 0)
+		(at 30.48 69.85 0)
 		(unit 1)
 		(body_style 1)
 		(exclude_from_sim no)
 		(in_bom yes)
-		(on_board yes)
+		(on_board no)
 		(in_pos_files yes)
 		(dnp no)
 		(property "Reference" "F1"
-			(at 61.722 104.14 0)
-			(show_name no)
-			(do_not_autoplace no)
-			(effects
-				(font
-					(size 1.27 1.27)
-				)
-			)
-		)
-		(property "Value" "5A (Micro2 blade)"
-			(at 60.96 91.948 0)
+			(at 29.972 73.66 0)
+			(show_name no)
+			(do_not_autoplace no)
+			(effects
+				(font
+					(size 1.27 1.27)
+				)
+			)
+		)
+		(property "Value" "5A Micro2, inline"
+			(at 29.21 61.468 0)
 			(show_name no)
 			(do_not_autoplace no)
@@
 		)
 		(property "Footprint" "Connector_PinHeader_2.54mm:PinHeader_1x02_P2.54mm_Vertical"
-			(at 62.23 100.33 0)
+			(at 30.48 69.85 0)
 			(hide yes)
 			(show_name no)
@@
 		)
 		(property "Datasheet" ""
-			(at 62.23 100.33 0)
+			(at 30.48 69.85 0)
 			(hide yes)
 			(show_name no)
@@
 		)
 		(property "Description" ""
-			(at 62.23 100.33 0)
+			(at 30.48 69.85 0)
 			(show_name no)
 			(do_not_autoplace no)
@@
 	(symbol
 		(lib_id "Irin:BATT_CONN")
-		(at 16.51 104.14 0)
+		(at 59.69 96.52 0)
 		(unit 1)
 		(body_style 1)
@@
 		(dnp no)
 		(property "Reference" "J1"
-			(at 20.32 102.87 0)
+			(at 63.5 95.25 0)
 			(show_name no)
 			(do_not_autoplace no)
@@
 		)
 		(property "Value" "Battery terminals"
-			(at 20.32 106.68 0)
+			(at 63.5 99.06 0)
 			(show_name no)
 			(do_not_autoplace no)
@@
 		)
 		(property "Footprint" "Connector_PinHeader_2.54mm:PinHeader_1x02_P2.54mm_Vertical"
-			(at 16.51 104.14 0)
+			(at 59.69 96.52 0)
 			(hide yes)
 			(show_name no)
@@
 		)
 		(property "Datasheet" ""
-			(at 16.51 104.14 0)
+			(at 59.69 96.52 0)
 			(hide yes)
 			(show_name no)
@@
 		)
 		(property "Description" ""
-			(at 16.51 104.14 0)
+			(at 59.69 96.52 0)
 			(show_name no)
 			(do_not_autoplace no)
@@
 					(unit 1)
 				)
+			)
+		)
+	)
+	(wire
+		(pts
+			(xy 16.51 83.82) (xy 16.51 69.85)
+		)
+		(stroke
+			(width 0)
+			(type default)
+		)
+	)
+	(wire
+		(pts
+			(xy 16.51 69.85) (xy 26.67 69.85)
+		)
+		(stroke
+			(width 0)
+			(type default)
+		)
+	)
+	(wire
+		(pts
+			(xy 16.51 93.98) (xy 16.51 158.75)
+		)
+		(stroke
+			(width 0)
+			(type default)
+		)
+	)
+	(wire
+		(pts
+			(xy 16.51 158.75) (xy 59.69 158.75)
+		)
+		(stroke
+			(width 0)
+			(type default)
+		)
+	)
+	(junction
+		(at 59.69 158.75)
+		(diameter 0)
+		(color 0 0 0 0)
+	)
+	(rectangle
+		(start 6.35 46.99)
+		(end 49.53 102.87)
+		(stroke
+			(width 0)
+			(type dash)
+		)
+		(fill
+			(type none)
+		)
+	)
+	(text "OFF-BOARD (vehicle harness)\nF1: inline holder, as close to the\nbattery + terminal as practical."
+		(exclude_from_sim no)
+		(at 8.89 50.8 0)
+		(effects
+			(font
+				(size 1.27 1.27)
+			)
+			(justify left top)
+		)
+	)
+	(symbol
+		(lib_id "Device:Battery")
+		(at 16.51 88.9 0)
+		(unit 1)
+		(body_style 1)
+		(exclude_from_sim no)
+		(in_bom no)
+		(on_board no)
+		(in_pos_files no)
+		(dnp no)
+		(property "Reference" "BT1"
+			(at 19.05 87.63 0)
+			(show_name no)
+			(do_not_autoplace no)
+			(effects
+				(font
+					(size 1.27 1.27)
+				)
+				(justify left)
+			)
+		)
+		(property "Value" "Vehicle 12V (flooded, 50Ah)"
+			(at 19.05 90.17 0)
+			(show_name no)
+			(do_not_autoplace no)
+			(effects
+				(font
+					(size 1.27 1.27)
+				)
+				(justify left)
+			)
+		)
+		(property "Footprint" ""
+			(at 16.51 88.9 0)
+			(show_name no)
+			(do_not_autoplace no)
+			(hide yes)
+			(effects
+				(font
+					(size 1.27 1.27)
+				)
+			)
+		)
+		(property "Datasheet" ""
+			(at 16.51 88.9 0)
+			(show_name no)
+			(do_not_autoplace no)
+			(hide yes)
+			(effects
+				(font
+					(size 1.27 1.27)
+				)
+			)
+		)
+		(property "Description" "The car's 12 V battery; off-board, shown for the harness"
+			(at 16.51 88.9 0)
+			(show_name no)
+			(do_not_autoplace no)
+			(hide yes)
+			(effects
+				(font
+					(size 1.27 1.27)
+				)
+			)
+		)
+		(pin "1"
+		)
+		(pin "2"
+		)
+		(instances
+			(project "irin"
+				(path "/097d63fa-dc7b-4932-a049-360b053b132d"
+					(reference "BT1")
+					(unit 1)
+				)

Commit message: Hardware rev B: screw-terminal J1, full silkscreen, D1 standard
- J1: 5.08 mm 2-pin screw terminal (Phoenix MKDS 1,5-2-5.08 footprint,
  KF301-2P fits) at the top edge, wire openings facing out; replaces the
  2.54 mm header, which neither takes 18 AWG nor survives vibration.
- Silkscreen for kit builders: part values on every part, J1 +/-, J2
  VCC/DATA/GND, U1 IN/OUT, U2 used pins and USB-C end, U3 pin names,
  "Irin - by AI7MG - rev B". Values shortened to fit (C1, J2, U3, J1).
  Mounting-hole references hidden.
- D1 (P6KE18A) fitted as standard: it also acts as the reverse-polarity
  crowbar (reversed hookup forward-biases D1 and blows F1). Schematic
  notes, CLAUDE.md, PARTS.md and README updated.
- DRC: 0 errors; one silkscreen-clearance warning where the USB-C mark
  meets U2's outline, intentionally. ERC: the 12 library-config warnings.

Co-Authored-By: Claude Opus 5.5 <noreply@anthropic.com>
Parts:
- C1: value 2nF mica (2x1000pF) -> 2nF mica
- D1: value P6KE18A (opt.) -> P6KE18A
- J1: value Battery terminals -> 12V IN; footprint Connector_PinHeader_2.54mm:PinHeader_1x02_P2.54mm_Vertical -> TerminalBlock_Phoenix:TerminalBlock_Phoenix_MKDS-1,5-2-5.08_1x02_P5.08mm_Horizontal
- J2: value DHT22 remote (VCC/DATA/GND) -> DHT22
- U3: value HiLetgo ADS1115 (0x48, ADDR->GND) -> ADS1115 (HiLetgo)
Other:
- note added: "No series reverse-polarity diode: D1 is the crowbar (reversed hookup blows F1). WS2812 RGB LED on U2 is disabled in firmware -- pure parasitic draw."
- note added: "TVS D1: P6KE18A, UNIDIRECTIONAL, fitted as standard. BANDED END (K, cathode, square pad) to PROT, A (anode) to GND. Reverse-biased in normal service: VRWM 15.3 V, breakdown 17.1-18.9 V, clamps a surge at Vc 25.2 V (MP1584 abs max 30 V). Fitted backwards it is a forward diode across the supply and blows F1. That is also the reverse-polarity protection: a reversed hookup forward-biases D1 and blows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"
- note removed: "Reverse-polarity protection deliberately omitted (owner-built, wired once). WS2812 RGB LED on U2 is disabled in firmware -- pure parasitic draw."
- note removed: "TVS D1: P6KE18A, UNIDIRECTIONAL, optional. BANDED END (K, cathode, square pad) to PROT, A (anode) to GND. Reverse-biased in normal service: VRWM 15.3 V, breakdown 17.1-18.9 V, clamps a surge at Vc 25.2 V (MP1584 abs max 30 V). Fitted backwards it is a forward diode across the supply and blows F1."
Changed lines of the file:
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@@
 		)
 	)
-	(text "TVS D1: P6KE18A, UNIDIRECTIONAL, optional.\nBANDED END (K, cathode, square pad) to PROT,\nA (anode) to GND.\nReverse-biased in normal service:\nVRWM 15.3 V, breakdown 17.1-18.9 V,\nclamps a surge at Vc 25.2 V (MP1584 abs max 30 V).\nFitted backwards it is a forward diode across\nthe supply and blows F1."
+	(text "TVS D1: P6KE18A, UNIDIRECTIONAL, fitted as standard.\nBANDED END (K, cathode, square pad) to PROT,\nA (anode) to GND.\nReverse-biased in normal service:\nVRWM 15.3 V, breakdown 17.1-18.9 V,\nclamps a surge at Vc 25.2 V (MP1584 abs max 30 V).\nFitted backwards it is a forward diode across\nthe supply and blows F1. That is also the\nreverse-polarity protection: a reversed hookup\nforward-biases D1 and blows F1 (crowbar)."
 		(exclude_from_sim no)
 		(at 22 130 0)
@@
 		)
 	)
-	(text "Reverse-polarity protection deliberately omitted (owner-built, wired once).\nWS2812 RGB LED on U2 is disabled in firmware -- pure parasitic draw."
+	(text "No series reverse-polarity diode: D1 is the crowbar (reversed hookup blows F1).\nWS2812 RGB LED on U2 is disabled in firmware -- pure parasitic draw."
 		(exclude_from_sim no)
 		(at 245 130 0)
@@
 			)
 		)
-		(property "Value" "P6KE18A (opt.)"
+		(property "Value" "P6KE18A"
 			(at 89.662 95.504 0)
 			(show_name no)
@@
 			)
 		)
-		(property "Value" "HiLetgo ADS1115 (0x48, ADDR->GND)"
+		(property "Value" "ADS1115 (HiLetgo)"
 			(at 373.38 43.942 0)
 			(show_name no)
@@
 			)
 		)
-		(property "Value" "DHT22 remote (VCC/DATA/GND)"
+		(property "Value" "DHT22"
 			(at 370.586 97.79 0)
 			(show_name no)
@@
 			)
 		)
-		(property "Value" "2nF mica (2x1000pF)"
+		(property "Value" "2nF mica"
 			(at 150.114 141.986 0)
 			(show_name no)
@@
 			)
 		)
-		(property "Value" "Battery terminals"
+		(property "Value" "12V IN"
 			(at 63.5 99.06 0)
 			(show_name no)
@@
 			)
 		)
-		(property "Footprint" "Connector_PinHeader_2.54mm:PinHeader_1x02_P2.54mm_Vertical"
+		(property "Footprint" "TerminalBlock_Phoenix:TerminalBlock_Phoenix_MKDS-1,5-2-5.08_1x02_P5.08mm_Horizontal"
 			(at 59.69 96.52 0)
 			(hide yes)
