File: hardware/irin.kicad_sch (KiCad schematic)
At the start: 13 parts, among them J1 12V IN, J2 DHT22, U1 MP1584EN set to 5.0V, U2 01Space ESP32-C3-0.42LCD, U3 ADS1115 (HiLetgo)

Commit message: Fix the U1 footprint; rev B's is 0.1in too narrow
The first rev B board was populated 2026-10-20 and the MP1584EN would not
fit U1. Built anyway by clipping one leg off each negative end and mounting
the module from the underside -- board #1 is live and reading 12.55 V and
14.40 V dead-on, with the breadboard's divider resistors transplanted so
the existing calibration carries over unchanged.

The old footprint's across-module spacing was ruler-measured at +/-0.5mm and
came out 0.1in too narrow overall: inner holes 0.2in apart where the part
needs 0.3in. Caliper measurement puts the four holes along an edge at
0.0 / 0.1 / 0.4 / 0.5 in, and the module outline at 0.66 x 0.86 in
(16.76 x 21.84 mm). The 0.7in row spacing was already right.

MP1584EN_HW133_2x2Pad_P2.54mm_W10.16mm_L17.78mm is the corrected footprint,
with a true measured outline rather than a placeholder box, and the
schematic now points at it. The old W7.62mm footprint is kept but marked
DEPRECATED in its own description, since the rev B boards were fabbed with
it.

The board file still carries the old embedded footprint: rev C needs
Update PCB from Schematic to pull this in, and a re-plot before fab.

Co-Authored-By: Claude Opus 5 <noreply@anthropic.com>
Parts:
- U1: footprint Irin:MP1584EN_HW133_2x2Pad_P2.54mm_W7.62mm_L17.78mm -> Irin:MP1584EN_HW133_2x2Pad_P2.54mm_W10.16mm_L17.78mm
Changed lines of the file:
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@@
 			)
 		)
-		(property "Footprint" "Irin:MP1584EN_HW133_2x2Pad_P2.54mm_W7.62mm_L17.78mm"
+		(property "Footprint" "Irin:MP1584EN_HW133_2x2Pad_P2.54mm_W10.16mm_L17.78mm"
 			(at 245.11 87.63 0)
 			(hide yes)
